Commit message: fix: vendor real AR4 (mk5) URDF + meshes, emit per-link poses
Three issues with the AR4 experiment in MICROROBOTICA, all rooted in
the same place: server.py had no idea how to map ``arm_link_<i>``,
``motor_rotor``, or ``magnet`` actor names to anything in the graph
state. They got silently skipped, all six arm-link Xforms stayed at
the USD origin, and the placeholder cubes overlapped at workspace
centre.

Changes:

* **Real AR4 mk5 URDF + STL meshes** vendored from the upstream
  Annin-Robotics/ar4_ros_driver ROS package (mk5 because its mesh dir
  matches the macro structure; mk3 mesh dir is incomplete on
  upstream). 22 visual STLs (~49 MB) baked via ``scene/_bake_meshes.py``
  into a single ``assets/ar4_meshes.usdc`` (35 MB binary USD) which
  ``world.usda`` references one Mesh-prim per arm link. Raw STLs are
  gitignored; ``assets/_fetch_meshes.py`` re-downloads them if you
  want to re-bake.

* **RobotArmNode now reports URDF link frames** (joint origins), not
  COM frames. ``update`` computes per-link world poses via
  ``joint_to_world_transforms`` and stores them in state under
  ``link_poses_world`` and ``end_effector_pose_world``, so visual
  meshes anchored to the URDF link frame land in the right place.
  ``compute_boundary_fluxes`` uses the same convention; XLA hoists
  the duplicate FK call inside the compiled gm.step.

* **server.py ``_state_to_result_frame``** resolves three composite
  actor name patterns to the right state lookups:
    * ``arm_link_<i>`` → ``state["arm"]["link_poses_world"][i]``
    * ``motor_rotor``  → ``state["motor"]["rotor_pose_world"]``
    * ``magnet``       → ``state["motor"]["rotor_pose_world"]``
  Plus a generic ``pose`` state-field shorthand that emits both
  position and orientation from a 7-vector. Backward-compatible:
  legacy ``position`` / ``orientation`` / ``field_vector`` paths
  are unchanged.

Verified end-to-end: AR4 home pose now spreads each link across the
arm's 47 cm reach, magnet sits 5 cm beyond the EE, microrobot at
vessel centre. Test fixture ``test_ee_pose_at_q_zero`` updated to
the new joint-frame convention (its ``EE_OFFSET`` was tuned for the
COM-frame regime).

10/10 RobotArm tests pass; 3-link planar fixture FK verified to
analytical < 1e-10 m; world.usda parses cleanly via OpenUSD (18
prims).

Co-Authored-By: Claude Opus 4.7 (1M context) <noreply@anthropic.com>

File: experiments/ar4_helical_drive/assets/ar4.urdf (robot description, URDF)
Before this commit: robot ar4, 8 links, 7 joints
Links:
- added link base_link_aluminum; visual mesh filename=meshes/ar4_mk5/Link_Base_Aluminum.STL
- added link base_link_enclosure; visual mesh filename=meshes/ar4_mk5/Link_Base_Enclosure.STL
- added link base_link_motor; visual mesh filename=meshes/ar4_mk5/Link_Base_Motor.STL
- added link ee_link
- added link link_1_aluminum; collision mesh filename=meshes/ar4_mk5/Link_1_Col.STL; visual mesh filename=meshes/ar4_mk5/Link_1_Aluminum.STL
- added link link_1_motor; visual mesh filename=meshes/ar4_mk5/Link_1_Motor.STL
- added link link_2_aluminum; collision mesh filename=meshes/ar4_mk5/Link_2_Col.STL; visual mesh filename=meshes/ar4_mk5/Link_2_Aluminum.STL
- added link link_2_cover; visual mesh filename=meshes/ar4_mk5/Link_2_Cover.STL
- added link link_2_logo; visual mesh filename=meshes/ar4_mk5/Link_2_Logo.STL
- added link link_2_motor; visual mesh filename=meshes/ar4_mk5/Link_2_Motor.STL
- added link link_3_aluminum; collision mesh filename=meshes/ar4_mk5/Link_3_Col.STL; visual mesh filename=meshes/ar4_mk5/Link_3_Aluminum.STL
- added link link_3_motor; visual mesh filename=meshes/ar4_mk5/Link_3_Motor.STL
- added link link_4_aluminum; collision mesh filename=meshes/ar4_mk5/Link_4_Col.STL; visual mesh filename=meshes/ar4_mk5/Link_4_Aluminum.STL
- added link link_4_cover; visual mesh filename=meshes/ar4_mk5/Link_4_Cover.STL
- added link link_4_logo; visual mesh filename=meshes/ar4_mk5/Link_4_Logo.STL
- added link link_4_motor; visual mesh filename=meshes/ar4_mk5/Link_4_Motor.STL
- added link link_5_aluminum; visual mesh filename=meshes/ar4_mk5/Link_5_Aluminum.STL
- added link link_5_motor; visual mesh filename=meshes/ar4_mk5/Link_5_Motor.STL
- added link link_6_aluminum; visual mesh filename=meshes/ar4_mk5/Link_6_Aluminum.STL
- link base_link: mass 3.0 -> 0.7102
- link link_1: mass 1.5 -> 0.88065
- link link_2: mass 1.8 -> 0.57738
- link link_3: mass 1.2 -> 0.1787
- link link_4: mass 0.5 -> 0.34936
- link link_5: mass 0.3 -> 0.11562
- link link_6: mass 0.2 -> 0.013863
Joints:
- removed joint world_to_base
- added joint base_joint: type fixed, parent world, child base_link, origin xyz=0 0 0 rpy=0 0 0
- added joint base_link_aluminum_joint: type fixed, parent base_link, child base_link_aluminum, origin xyz=0 0 0 rpy=0 0 0
- added joint base_link_enclosure_joint: type fixed, parent base_link, child base_link_enclosure, origin xyz=0 0 0 rpy=0 0 0
- added joint base_link_motor_joint: type fixed, parent base_link, child base_link_motor, origin xyz=0 0 0 rpy=0 0 0
- added joint ee_joint: type fixed, parent link_6, child ee_link, origin xyz=0 0 0 rpy=0 0 0
- added joint link_1_aluminum_joint: type fixed, parent link_1, child link_1_aluminum, origin xyz=0 0 0 rpy=0 0 0
- added joint link_1_motor_joint: type fixed, parent link_1, child link_1_motor, origin xyz=0 0 0 rpy=0 0 0
- added joint link_2_aluminum_joint: type fixed, parent link_2, child link_2_aluminum, origin xyz=0 0 0 rpy=0 0 0
- added joint link_2_cover_joint: type fixed, parent link_2, child link_2_cover, origin xyz=0 0 0 rpy=0 0 0
- added joint link_2_logo_joint: type fixed, parent link_2, child link_2_logo, origin xyz=0 0 0 rpy=0 0 0
- added joint link_2_motor_joint: type fixed, parent link_2, child link_2_motor, origin xyz=0 0 0 rpy=0 0 0
- added joint link_3_aluminum_joint: type fixed, parent link_3, child link_3_aluminum, origin xyz=0 0 0 rpy=0 0 0
- added joint link_3_motor_joint: type fixed, parent link_3, child link_3_motor, origin xyz=0 0 0 rpy=0 0 0
- added joint link_4_aluminum_joint: type fixed, parent link_4, child link_4_aluminum, origin xyz=0 0 0 rpy=0 0 0
- added joint link_4_cover_joint: type fixed, parent link_4, child link_4_cover, origin xyz=0 0 0 rpy=0 0 0
- added joint link_4_logo_joint: type fixed, parent link_4, child link_4_logo, origin xyz=0 0 0 rpy=0 0 0
- added joint link_4_motor_joint: type fixed, parent link_4, child link_4_motor, origin xyz=0 0 0 rpy=0 0 0
- added joint link_5_aluminum_joint: type fixed, parent link_5, child link_5_aluminum, origin xyz=0 0 0 rpy=0 0 0
- added joint link_5_motor_joint: type fixed, parent link_5, child link_5_motor, origin xyz=0 0 0 rpy=0 0 0
- added joint link_6_aluminum_joint: type fixed, parent link_6, child link_6_aluminum, origin xyz=0 0 0 rpy=0 0 0
- joint joint_1: limit lower=-2.967 upper=2.967 effort=50 velocity=3.14 -> lower=-2.792526803190927 upper=2.792526803190927 effort=-1 velocity=1.0472; origin xyz=0 0 0.169 rpy=0 0 0 -> xyz=0 0 0.092 rpy=3.141592653589793 0 0
- joint joint_2: axis 0 1 0 -> 0 0 -1; limit lower=-1.571 upper=1.571 effort=50 velocity=3.14 -> lower=-0.7330382858376184 upper=1.5707963267948966 effort=-1 velocity=1.0472; origin xyz=0 0 0.10 rpy=0 0 0 -> xyz=0 0.06415 -0.07778 rpy=1.5708 0 -1.5708
- joint joint_3: axis 0 1 0 -> 0 0 -1; limit lower=-2.548 upper=2.548 effort=40 velocity=3.14 -> lower=-1.5533430342749532 upper=0.9075712110370514 effort=-1 velocity=1.0472; origin xyz=0.305 0 0 rpy=0 0 0 -> xyz=0 -0.305 0 rpy=0 0 3.1416
- joint joint_4: axis 1 0 0 -> 0 0 -1; limit lower=-2.967 upper=2.967 effort=20 velocity=6.28 -> lower=-3.141592653589793 upper=3.141592653589793 effort=-1 velocity=1.0472; origin xyz=0.264 0 0 rpy=0 0 0 -> xyz=0 0 0 rpy=1.5708 0 -1.5708
- joint joint_5: axis 0 1 0 -> 1 0 0; limit lower=-1.833 upper=1.833 effort=20 velocity=6.28 -> lower=-1.8325957145940461 upper=1.8325957145940461 effort=-1 velocity=1.0472; origin xyz=0.064 0 0 rpy=0 0 0 -> xyz=0 0 -0.22294 rpy=3.141592653589793 0 -1.5708
- joint joint_6: axis 1 0 0 -> 0 0 1; limit lower=-3.1416 upper=3.1416 effort=20 velocity=6.28 -> lower=-3.141592653589793 upper=3.141592653589793 effort=-1 velocity=1.5708; origin xyz=0 0 0 rpy=0 0 0 -> xyz=0 0 0.041 rpy=0 0 0
